File: hardware/kicad/in18_nixie_clock/esp32.kicad_sch (KiCad schematic)
At the start: 0 parts

Commit message: Add several schematics
Parts:
- added C10, C11, C7, C8: 10u 35v, Capacitor_SMD:C_0805_2012Metric, symbol Device:C
- added C12, C9: 100n, Capacitor_SMD:C_0402_1005Metric, symbol Device:C
- added J2: USB_B_Micro, USB_conn_user:USB_Micro-B_EDAC_UCON00686, symbol Connector:USB_B_Micro
- added Q2, Q3: SS8050-G, BJT_user:SOT95P240X115-3N, symbol BJT_user:SS8050-G
- added R3: 2K, Resistor_SMD:R_0805_2012Metric_Pad1.20x1.40mm_HandSolder, symbol Device:R
- added R4, R5: 12K, Resistor_SMD:R_0805_2012Metric_Pad1.20x1.40mm_HandSolder, symbol Device:R
- added R6, R7, R8, R9: 0, Resistor_SMD:R_0805_2012Metric_Pad1.20x1.40mm_HandSolder, symbol Device:R
- added TP1: VBUS, TestPoint:TestPoint_Pad_D2.0mm, symbol Connector:TestPoint
- added TP10: DTR, TestPoint:TestPoint_Pad_D2.0mm, symbol Connector:TestPoint
- added TP11: RTS, TestPoint:TestPoint_Pad_D2.0mm, symbol Connector:TestPoint
- added TP2: TX, TestPoint:TestPoint_Pad_D2.0mm, symbol Connector:TestPoint
- added TP3: RX, TestPoint:TestPoint_Pad_D2.0mm, symbol Connector:TestPoint
- added TP4: CTS, TestPoint:TestPoint_Pad_D2.0mm, symbol Connector:TestPoint
- added TP5: DSR, TestPoint:TestPoint_Pad_D2.0mm, symbol Connector:TestPoint
- added TP6: DCD, TestPoint:TestPoint_Pad_D2.0mm, symbol Connector:TestPoint
- added TP7: RI, TestPoint:TestPoint_Pad_D2.0mm, symbol Connector:TestPoint
- added TP8: PROG_EN, TestPoint:TestPoint_Pad_D2.0mm, symbol Connector:TestPoint
- added TP9: ESP_EN, TestPoint:TestPoint_Pad_D2.0mm, symbol Connector:TestPoint
- added U2: IP4220CZ6F, ESD_user:SOT95P275X110-6N, symbol ESD_user:IP4220CZ6F
- added U3: ESP32-WROOM-32, RF_Module:ESP32-WROOM-32, symbol RF_Module:ESP32-WROOM-32
- added U4: CP2102N-Axx-xQFN28, Package_DFN_QFN:QFN-28-1EP_5x5mm_P0.5mm_EP3.35x3.35mm, symbol Interface_USB:CP2102N-Axx-xQFN28
Connections:
- new net: Q2.1, R4.1
- new net: TP5.1, U4.27 (~{DSR})
- new net: TP6.1, U4.1 (~{DCD})
- new net: TP7.1, U4.2 (~{RI}/CLK)
- new net: Q3.1, R5.1
- new net: R3.2, U4.9 (~{RST})
- new net +3V3: C10.1, C11.1, C12.1, C7.1, C8.1, C9.1, R3.1, U3.2 (VDD), U4.6 (VDD), U4.7 (VREGIN)
- new net CTS: TP4.1, U4.23 (~{CTS})
- new net D+: J2.3 (D+), U2.3 (I/O_2), U4.4 (D+)
- new net D-: J2.2 (D-), U2.1 (I/O_1), U4.5 (D-)
- new net DTR: Q2.2, R5.2, TP10.1, U4.28 (~{DTR})
- new net ESP_EN: Q3.3, TP9.1, U3.3 (EN)
- new net ESP_RX: R6.2, R7.2, U3.34 (RXD0/IO3)
- new net ESP_TX: R8.2, R9.2, U3.35 (TXD0/IO1)
- new net GND: C10.2, C11.2, C12.2, C7.2, C8.2, C9.2, J2.5 (GND), J2.6 (Shield), U2.2 (GND), U3.1 (GND), U3.15 (GND), U3.38 (GND), U3.39 (GND), U4.29 (GND), U4.3 (GND)
- new net PROG_EN: Q2.3, TP8.1, U3.25 (IO0)
- new net RTS: Q3.2, R4.2, TP11.1, U4.24 (~{RTS})
- new net RXD: R7.1, R9.1, TP3.1, U4.25 (RXD)
- new net TXD: R6.1, R8.1, TP2.1, U4.26 (TXD)
- new net VBUS: J2.1 (VBUS), TP1.1, U2.5 (VP), U4.8 (VBUS)
- no-connect marks 0 -> 17
Other:
- note added: "DNP"
- note added: "ESD protection"
- note added: "GPIO: 24 --> nixie driver 12 --> nixie driver with duplex 6 --> nixie PWM 2 --> uart TXRX 1 --> RGB leds Total IO required: 33 without duplex 21 with duplex"
- note added: "Put ESP automatically in UART programming mode"
- note added: "TX --> RX RX <-- TX If RX, TX are crossed: Remove R9 and R10 Place R8 and R11"
- note added: "USB to serial converter"
