File: hardware/kicad/in18_nixie_clock/in18_nixie_clock.kicad_pcb (KiCad board)
At the start: 0 parts

Commit message: Add several schematics
Parts:
- added C1: 100nF, Capacitor_SMD:C_0805_2012Metric_Pad1.18x1.45mm_HandSolder, F.Cu at (428.2, 158.2)
- added C10: 10u 35v, Capacitor_SMD:C_0805_2012Metric, F.Cu at (369.2, 184.6)
- added C11: 10u 35v, Capacitor_SMD:C_0805_2012Metric, F.Cu at (402.2, 152.0)
- added C12: 100n, Capacitor_SMD:C_0402_1005Metric, F.Cu at (363.6, 187.0)
- added C13: 100n, Capacitor_SMD:C_0402_1005Metric, F.Cu at (487.6, 91.2)
- added C14: 100n, Capacitor_SMD:C_0402_1005Metric, F.Cu at (490.5, 89.3)
- added C15: 100n, Capacitor_SMD:C_0402_1005Metric, F.Cu at (484.8, 91.2)
- added C16: 100n, Capacitor_SMD:C_0402_1005Metric, F.Cu at (493.4, 89.3)
- added C17: 100n, Capacitor_SMD:C_0402_1005Metric, F.Cu at (484.8, 89.3)
- added C18: 100n, Capacitor_SMD:C_0402_1005Metric, F.Cu at (487.6, 89.3)
- added C19: 100n, Capacitor_SMD:C_0402_1005Metric, F.Cu at (421.1, 138.5)
- added C2: 100nF, Capacitor_SMD:C_0805_2012Metric_Pad1.18x1.45mm_HandSolder, F.Cu at (430.9, 152.0)
- added C20: 100n, Capacitor_SMD:C_0402_1005Metric, F.Cu at (430.6, 131.1)
- added C21: 100n, Capacitor_SMD:C_0402_1005Metric, F.Cu at (371.4, 59.3)
- added C5: 100nF, 250V, Capacitor_SMD:C_0805_2012Metric_Pad1.18x1.45mm_HandSolder, F.Cu at (430.9, 155.1)
- added C7: 10u 35v, Capacitor_SMD:C_0805_2012Metric, F.Cu at (390.5, 163.0)
- added C8: 10u 35v, Capacitor_SMD:C_0805_2012Metric, F.Cu at (388.0, 167.3)
- added C9: 100n, Capacitor_SMD:C_0402_1005Metric, F.Cu at (366.5, 187.1)
- added D2: WS2812B, LED_SMD:LED_WS2812B_PLCC4_5.0x5.0mm_P3.2mm, F.Cu at (360.0, 90.0)
- added D3: WS2812B, LED_SMD:LED_WS2812B_PLCC4_5.0x5.0mm_P3.2mm, F.Cu at (487.5, 85.0)
- added D4: WS2812B, LED_SMD:LED_WS2812B_PLCC4_5.0x5.0mm_P3.2mm, F.Cu at (495.9, 85.0)
- added D5: WS2812B, LED_SMD:LED_WS2812B_PLCC4_5.0x5.0mm_P3.2mm, F.Cu at (495.9, 78.4)
- added D6: WS2812B, LED_SMD:LED_WS2812B_PLCC4_5.0x5.0mm_P3.2mm, F.Cu at (504.4, 78.4)
- added D7: WS2812B, LED_SMD:LED_WS2812B_PLCC4_5.0x5.0mm_P3.2mm, F.Cu at (504.4, 85.0)
- added J1: USB_B_Micro, USB_conn_user:USB_Micro-B_EDAC_UCON00686, F.Cu at (385.7, 155.5)
- added J2: USB_B_Micro, USB_conn_user:USB_Micro-B_EDAC_UCON00686, F.Cu at (467.3, 117.0)
- added N1: IN18, Nixie_tubes:nixies-us-IN-18-DSUB, F.Cu at (360.0, 90.0)
- added N2: IN18, Nixie_tubes:nixies-us-IN-18-DSUB, F.Cu at (367.4, 41.9)
- added Q1: IRF644PBF, FET_user:TO254P465X1024X2050-3P, F.Cu at (420.0, 154.5)
- added Q10: MPSA92, Package_TO_SOT_THT:TO-92_Inline, F.Cu at (441.3, 127.0)
- added Q11: MPSA42, Package_TO_SOT_THT:TO-92_Inline, F.Cu at (434.8, 127.0)
- added Q12: MPSA42, Package_TO_SOT_THT:TO-92_Inline, F.Cu at (430.2, 121.1)
- added Q13: MPSA42, Package_TO_SOT_THT:TO-92_Inline, F.Cu at (430.2, 115.3)
- added Q14: MPSA42, Package_TO_SOT_THT:TO-92_Inline, F.Cu at (436.7, 115.3)
- added Q15: MPSA42, Package_TO_SOT_THT:TO-92_Inline, F.Cu at (421.6, 127.6)
- added Q16: MPSA42, Package_TO_SOT_THT:TO-92_Inline, F.Cu at (385.8, 58.3)
- added Q17: MPSA42, Package_TO_SOT_THT:TO-92_Inline, F.Cu at (394.4, 34.5)
- added Q18: MPSA42, Package_TO_SOT_THT:TO-92_Inline, F.Cu at (407.5, 28.7)
- added Q19: MPSA42, Package_TO_SOT_THT:TO-92_Inline, F.Cu at (392.4, 40.9)
- added Q2: SS8050-G, BJT_user:SOT95P240X115-3N, F.Cu at (392.8, 152.8)
- added Q20: MPSA42, Package_TO_SOT_THT:TO-92_Inline, F.Cu at (385.8, 52.5)
- added Q21: MPSA42, Package_TO_SOT_THT:TO-92_Inline, F.Cu at (392.4, 46.7)
- added Q22: MPSA92, Package_TO_SOT_THT:TO-92_Inline, F.Cu at (399.0, 40.3)
- added Q23: MPSA42, Package_TO_SOT_THT:TO-92_Inline, F.Cu at (400.9, 34.5)
- added Q24: MPSA42, Package_TO_SOT_THT:TO-92_Inline, F.Cu at (400.9, 28.7)
- added Q25: MPSA42, Package_TO_SOT_THT:TO-92_Inline, F.Cu at (394.4, 28.7)
- added Q26: MPSA42, Package_TO_SOT_THT:TO-92_Inline, F.Cu at (385.8, 46.7)
- added Q27: MPSA42, Package_TO_SOT_THT:TO-92_Inline, F.Cu at (385.8, 40.9)
- added Q3: SS8050-G, BJT_user:SOT95P240X115-3N, F.Cu at (359.8, 185.4)
- added Q4: MPSA42, Package_TO_SOT_THT:TO-92_Inline, F.Cu at (449.9, 121.1)
- added Q5: MPSA42, Package_TO_SOT_THT:TO-92_Inline, F.Cu at (428.2, 127.6)
- added Q6: MPSA42, Package_TO_SOT_THT:TO-92_Inline, F.Cu at (443.3, 121.1)
- added Q7: MPSA42, Package_TO_SOT_THT:TO-92_Inline, F.Cu at (436.7, 121.1)
- added Q8: MPSA42, Package_TO_SOT_THT:TO-92_Inline, F.Cu at (443.3, 115.3)
- added Q9: MPSA42, Package_TO_SOT_THT:TO-92_Inline, F.Cu at (449.9, 115.3)
- added R10: 10K, Resistor_SMD:R_0805_2012Metric_Pad1.20x1.40mm_HandSolder, F.Cu at (426.7, 131.6)
- added R11: 10K, Resistor_SMD:R_0805_2012Metric_Pad1.20x1.40mm_HandSolder, F.Cu at (435.1, 131.0)
- added R12: 10K, Resistor_SMD:R_0805_2012Metric_Pad1.20x1.40mm_HandSolder, F.Cu at (422.0, 131.6)
- added R13: 33k, Resistor_SMD:R_0805_2012Metric_Pad1.20x1.40mm_HandSolder, F.Cu at (456.8, 113.5)
- added R14: 10K, Resistor_SMD:R_0805_2012Metric_Pad1.20x1.40mm_HandSolder, F.Cu at (358.1, 59.8)
- added R15: 100K, Resistor_SMD:R_0805_2012Metric_Pad1.20x1.40mm_HandSolder, F.Cu at (362.8, 59.8)
- added R16: 470K, Resistor_SMD:R_0805_2012Metric_Pad1.20x1.40mm_HandSolder, F.Cu at (353.3, 59.8)
- added R17: 10K, Resistor_SMD:R_0805_2012Metric_Pad1.20x1.40mm_HandSolder, F.Cu at (367.6, 59.8)
- added R18: 33k, Resistor_SMD:R_0805_2012Metric_Pad1.20x1.40mm_HandSolder, F.Cu at (483.8, 36.3)
- added R19: 10K, Resistor_SMD:R_0805_2012Metric_Pad1.20x1.40mm_HandSolder, F.Cu at (483.8, 33.3)
- added R20: 10K, Resistor_SMD:R_0805_2012Metric_Pad1.20x1.40mm_HandSolder, F.Cu at (479.0, 33.3)
- added R21: 10K, Resistor_SMD:R_0805_2012Metric_Pad1.20x1.40mm_HandSolder, F.Cu at (488.5, 33.3)
- added R22: 10K, Resistor_SMD:R_0805_2012Metric_Pad1.20x1.40mm_HandSolder, F.Cu at (479.0, 36.3)
- added R23: 10K, Resistor_SMD:R_0805_2012Metric_Pad1.20x1.40mm_HandSolder, F.Cu at (488.5, 36.3)
- added R24: 10K, Resistor_SMD:R_0805_2012Metric_Pad1.20x1.40mm_HandSolder, F.Cu at (463.1, 42.2)
- added R25: 10K, Resistor_SMD:R_0805_2012Metric_Pad1.20x1.40mm_HandSolder, F.Cu at (463.1, 33.3)
- added R26: 10K, Resistor_SMD:R_0805_2012Metric_Pad1.20x1.40mm_HandSolder, F.Cu at (453.6, 33.3)
- added R27: 33k, Resistor_SMD:R_0805_2012Metric_Pad1.20x1.40mm_HandSolder, F.Cu at (458.4, 33.3)
- added R28: 10K, Resistor_SMD:R_0805_2012Metric_Pad1.20x1.40mm_HandSolder, F.Cu at (453.6, 42.2)
- added R29: 100K, Resistor_SMD:R_0805_2012Metric_Pad1.20x1.40mm_HandSolder, F.Cu at (453.6, 39.2)
- added R3: 2K, Resistor_SMD:R_0805_2012Metric_Pad1.20x1.40mm_HandSolder, F.Cu at (392.8, 156.6)
- added R30: 470K, Resistor_SMD:R_0805_2012Metric_Pad1.20x1.40mm_HandSolder, F.Cu at (453.6, 36.3)
- added R31: 10K, Resistor_SMD:R_0805_2012Metric_Pad1.20x1.40mm_HandSolder, F.Cu at (463.1, 39.2)
- added R32: 33k, Resistor_SMD:R_0805_2012Metric_Pad1.20x1.40mm_HandSolder, F.Cu at (467.9, 33.3)
- added R33: 10K, Resistor_SMD:R_0805_2012Metric_Pad1.20x1.40mm_HandSolder, F.Cu at (463.1, 36.3)
- added R34: 10K, Resistor_SMD:R_0805_2012Metric_Pad1.20x1.40mm_HandSolder, F.Cu at (458.4, 36.3)
- added R35: 10K, Resistor_SMD:R_0805_2012Metric_Pad1.20x1.40mm_HandSolder, F.Cu at (458.4, 42.2)
- added R36: 10K, Resistor_SMD:R_0805_2012Metric_Pad1.20x1.40mm_HandSolder, F.Cu at (458.4, 39.2)
- added R37: 10K, Resistor_SMD:R_0805_2012Metric_Pad1.20x1.40mm_HandSolder, F.Cu at (467.9, 36.3)
- added R4: 12K, Resistor_SMD:R_0805_2012Metric_Pad1.20x1.40mm_HandSolder, F.Cu at (364.6, 184.6)
- added R5: 12K, Resistor_SMD:R_0805_2012Metric_Pad1.20x1.40mm_HandSolder, F.Cu at (397.6, 155.0)
- added R6: 0, Resistor_SMD:R_0805_2012Metric_Pad1.20x1.40mm_HandSolder, F.Cu at (383.4, 167.2)
- added R7: 0, Resistor_SMD:R_0805_2012Metric_Pad1.20x1.40mm_HandSolder, F.Cu at (397.6, 152.0)
- added R8: 0, Resistor_SMD:R_0805_2012Metric_Pad1.20x1.40mm_HandSolder, F.Cu at (383.4, 170.2)
- added R9: 0, Resistor_SMD:R_0805_2012Metric_Pad1.20x1.40mm_HandSolder, F.Cu at (390.6, 160.0)
- added TP1: VBUS, TestPoint:TestPoint_Pad_D2.0mm, F.Cu at (399.1, 159.6)
- added TP10: DTR, TestPoint:TestPoint_Pad_D2.0mm, F.Cu at (373.4, 185.1)
- added TP11: RTS, TestPoint:TestPoint_Pad_D2.0mm, F.Cu at (387.1, 174.9)
- added TP2: TX, TestPoint:TestPoint_Pad_D2.0mm, F.Cu at (406.5, 152.6)
- added TP3: RX, TestPoint:TestPoint_Pad_D2.0mm, F.Cu at (392.2, 166.5)
- added TP4: CTS, TestPoint:TestPoint_Pad_D2.0mm, F.Cu at (387.8, 170.8)
- added TP5: DSR, TestPoint:TestPoint_Pad_D2.0mm, F.Cu at (395.0, 160.1)
- added TP6: DCD, TestPoint:TestPoint_Pad_D2.0mm, F.Cu at (383.0, 173.7)
- added TP7: RI, TestPoint:TestPoint_Pad_D2.0mm, F.Cu at (402.0, 155.6)
- added TP8: PROG_EN, TestPoint:TestPoint_Pad_D2.0mm, F.Cu at (383.0, 177.7)
- added TP9: ESP_EN, TestPoint:TestPoint_Pad_D2.0mm, F.Cu at (377.5, 185.1)
- added U1: MAX1771CSA+, Regulator_user:SOIC127P600X175-8N, F.Cu at (421.6, 160.0)
- added U2: IP4220CZ6F, ESD_user:SOT95P275X110-6N, F.Cu at (354.7, 185.3)
- added U3: ESP32-WROOM-32, RF_Module:ESP32-WROOM-32, F.Cu at (366.2, 172.1)
- added U4: CP2102N-Axx-xQFN28, Package_DFN_QFN:QFN-28-1EP_5x5mm_P0.5mm_EP3.35x3.35mm, F.Cu at (384.6, 162.1)
- added U5: PCF8574TS, Package_SO:SSOP-20_4.4x6.5mm_P0.65mm, F.Cu at (466.8, 127.7)
- added U6: 74HC42D,652, Logic_user:SOIC127P600X175-16N, F.Cu at (424.2, 118.7)
- added U7: 74HC42D,652, Logic_user:SOIC127P600X175-16N, F.Cu at (388.4, 32.1)
Other:
- copper layers 0 -> 2
