File: hardware/kicad/in18_nixie_clock/in18_nixies.kicad_sch (KiCad schematic)
At the start: 0 parts

Commit message: Add several schematics
Parts:
- added C13: 100n, Capacitor_SMD:C_0402_1005Metric, symbol Device:C
- added R?: 10K, Resistor_SMD:R_0805_2012Metric_Pad1.20x1.40mm_HandSolder, symbol Device:R
- added U5: PCF8574TS, Package_SO:SSOP-20_4.4x6.5mm_P0.65mm, symbol Interface_Expansion:PCF8574TS
Connections:
- new net: R?.1, U5.1 (~{INT})
- new net +3V3: C13.1, R?.2, U5.5 (VDD)
- new net A0_H_LS: U5.10 (P0), U5.16 (P4)
- new net A1_H_LS: U5.11 (P1), U5.17 (P5)
- new net A2_H_LS: U5.12 (P2), U5.19 (P6)
- new net A3_H_LS: U5.14 (P3), U5.20 (P7)
- new net GND: C13.2, U5.15 (VSS), U5.6 (A0), U5.7 (A1), U5.9 (A2)
- new net SCL: U5.2 (SCL)
- new net SDA: U5.4 (SDA)
Other:
- added sheet Nixie hour, least significant (nixie_h_ls.kicad_sch)
- added sheet Nixie hour, most significant (nixie_h_ms.kicad_sch)
- note added: "Hours"
